File: jack.sch (EAGLE design)
At the start: 35 parts, among them IC1 NUF2221W1T2G, IC2 ATSAMD21G18, IC3 LDO, J1 USB-micro, SW1 SPST3.5X6MM, X1 CX-3225 12.288MHz

Commit message: Minor changes (added BOM)
Parts:
- C10: value 100nF -> 10uF
- C4: device rcl:C-EUC0402K -> jack:C-EU
Changed lines of the file:
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@@
 <part name="C2" library="jack" deviceset="C-EU" device="" value="100nF"/>
 <part name="C3" library="jack" deviceset="C-EU" device="" value="100nF"/>
-<part name="C4" library="rcl" deviceset="C-EU" device="C0402K" value="100nF"/>
+<part name="C4" library="jack" deviceset="C-EU" device="" value="100nF"/>
 <part name="C5" library="jack" deviceset="C-EU" device="" value="100nF"/>
 <part name="VDD1" library="jack" deviceset="VDD" device=""/>
@@
 <part name="VBUS2" library="jack" deviceset="VBUS" device=""/>
 <part name="GND8" library="cortexm0" deviceset="GND" device=""/>
-<part name="C10" library="jack" deviceset="CPOL-EU" device="" value="100nF"/>
+<part name="C10" library="jack" deviceset="CPOL-EU" device="" value="10uF"/>
 <part name="C11" library="jack" deviceset="CPOL-EU" device="" value="10uF"/>
 <part name="X1" library="jack" deviceset="XTAL" device="CX-3225" value="CX-3225 12.288MHz"/>

Commit message: Updated .sch and .brd to match changes in library files
Ops, I forgot to save and close the project before pushing the last
commit :grin:
Parts:
- C10, C11, C6, C7: device jack:CPOL-EU -> jack:CPOL-EUCT3216
Changed lines of the file:
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@@
 <part name="GND3" library="cortexm0" deviceset="GND" device=""/>
 <part name="GND4" library="cortexm0" deviceset="GND" device=""/>
-<part name="C6" library="jack" deviceset="CPOL-EU" device="" value="10uF"/>
+<part name="C6" library="jack" deviceset="CPOL-EU" device="CT3216" value="10uF"/>
 <part name="VDD2" library="jack" deviceset="VDD" device=""/>
-<part name="C7" library="jack" deviceset="CPOL-EU" device="" value="10uF"/>
+<part name="C7" library="jack" deviceset="CPOL-EU" device="CT3216" value="10uF"/>
 <part name="GND5" library="cortexm0" deviceset="GND" device=""/>
 <part name="L1" library="jack" deviceset="L" device="" value="BLM18EG221"/>
@@
 <part name="VBUS2" library="jack" deviceset="VBUS" device=""/>
 <part name="GND8" library="cortexm0" deviceset="GND" device=""/>
-<part name="C10" library="jack" deviceset="CPOL-EU" device="" value="10uF"/>
-<part name="C11" library="jack" deviceset="CPOL-EU" device="" value="10uF"/>
+<part name="C10" library="jack" deviceset="CPOL-EU" device="CT3216" value="10uF"/>
+<part name="C11" library="jack" deviceset="CPOL-EU" device="CT3216" value="10uF"/>
 <part name="X1" library="jack" deviceset="XTAL" device="CX-3225" value="CX-3225 12.288MHz"/>
 <part name="C12" library="jack" deviceset="C-EU" device="" value="15pF"/>

Commit message: :feelsgood: Added BOM, Gerbers, 3D model and render
Parts:
- D1, D2: EAGLEUP (none) -> SOD323
- IC1: EAGLEUP (none) -> SOT363
- IC3: EAGLEUP (none) -> SOT223
- L1: EAGLEUP (none) -> R0603
- L2: EAGLEUP (none) -> ELLVFG
- R5: value 90 -> 68
- SW1: EAGLEUP (none) -> MOM-1181
- X1: EAGLEUP (none) -> CX3225
Changed lines of the file:
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@@
 <setting verticaltext="up"/>
 </settings>
-<grid distance="0.05" unitdist="inch" unit="inch" style="lines" multiple="1" display="no" altdistance="0.01" altunitdist="inch" altunit="inch"/>
+<grid distance="0.1" unitdist="inch" unit="inch" style="lines" multiple="1" display="no" altdistance="0.01" altunitdist="inch" altunit="inch"/>
 <layers>
 <layer number="1" name="Top" color="4" fill="1" visible="no" active="no"/>
@@
 <layer number="49" name="Reference" color="7" fill="1" visible="no" active="no"/>
 <layer number="50" name="dxf" color="7" fill="1" visible="no" active="no"/>
-<layer number="51" name="tDocu" color="7" fill="1" visible="no" active="no"/>
+<layer number="51" name="tDocu" color="15" fill="1" visible="no" active="no"/>
 <layer number="52" name="bDocu" color="7" fill="1" visible="no" active="no"/>
 <layer number="53" name="tGND_GNDA" color="7" fill="1" visible="no" active="no"/>
@@
 <part name="C7" library="jack" deviceset="CPOL-EU" device="CT3216" value="10uF"/>
 <part name="GND5" library="cortexm0" deviceset="GND" device=""/>
-<part name="L1" library="jack" deviceset="L" device="" value="BLM18EG221"/>
-<part name="L2" library="Panasonic-ELL" deviceset="ELL" device="-VXG" technology="VFG100MC" value="10UH"/>
+<part name="L1" library="jack" deviceset="L" device="" value="BLM18EG221">
+<attribute name="EAGLEUP" value="R0603"/>
+</part>
+<part name="L2" library="Panasonic-ELL" deviceset="ELL" device="-VXG" technology="VFG100MC" value="10UH">
+<attribute name="EAGLEUP" value="ELLVFG"/>
+</part>
 <part name="J1" library="Molex-47346-0001" deviceset="47346-0001" device="" value="USB-micro"/>
 <part name="C8" library="jack" deviceset="C-EU" device="" value="4.5nF"/>
 <part name="R1" library="jack" deviceset="R-EU" device="" value="1M"/>
-<part name="IC1" library="jack" deviceset="NUF2221W1T2G" device=""/>
+<part name="IC1" library="jack" deviceset="NUF2221W1T2G" device="">
+<attribute name="EAGLEUP" value="SOT363"/>
+</part>
 <part name="GND6" library="cortexm0" deviceset="GND" device=""/>
 <part name="C9" library="jack" deviceset="C-EU" device="" value="100nF"/>
@@
 <part name="R2" library="jack" deviceset="R-EU" device="" value="330"/>
 <part name="R3" library="jack" deviceset="R-EU" device="" value="10K"/>
-<part name="SW1" library="jack" deviceset="SPST" device="3.5X6MM"/>
-<part name="IC3" library="jack" deviceset="LDO" device=""/>
+<part name="SW1" library="jack" deviceset="SPST" device="3.5X6MM">
+<attribute name="EAGLEUP" value="MOM-1181"/>
+</part>
+<part name="IC3" library="jack" deviceset="LDO" device="">
+<attribute name="EAGLEUP" value="SOT223"/>
+</part>
 <part name="VDD4" library="jack" deviceset="VDD" device=""/>
 <part name="VBUS2" library="jack" deviceset="VBUS" device=""/>
@@
 <part name="C10" library="jack" deviceset="CPOL-EU" device="CT3216" value="10uF"/>
 <part name="C11" library="jack" deviceset="CPOL-EU" device="CT3216" value="10uF"/>
-<part name="X1" library="jack" deviceset="XTAL" device="CX-3225" value="CX-3225 12.288MHz"/>
+<part name="X1" library="jack" deviceset="XTAL" device="CX-3225" value="CX-3225 12.288MHz">
+<attribute name="EAGLEUP" value="CX3225"/>
+</part>
 <part name="C12" library="jack" deviceset="C-EU" device="" value="15pF"/>
 <part name="C13" library="jack" deviceset="C-EU" device="" value="15pF"/>
 <part name="GND9" library="cortexm0" deviceset="GND" device=""/>
-<part name="D1" library="diode" deviceset="BAT60J" device=""/>
-<part name="D2" library="diode" deviceset="BAT60J" device=""/>
+<part name="D1" library="diode" deviceset="BAT60J" device="">
+<attribute name="EAGLEUP" value="SOD323"/>
+</part>
+<part name="D2" library="diode" deviceset="BAT60J" device="">
+<attribute name="EAGLEUP" value="SOD323"/>
+</part>
 <part name="U$1" library="jack" deviceset="AGND" device=""/>
 <part name="VDD5" library="jack" deviceset="VDD" device=""/>
@@
 <part name="U$6" library="jack" deviceset="OSHW-LOGO" device=""/>
 <part name="D3" library="jack" deviceset="LED" device=""/>
-<part name="R5" library="jack" deviceset="R-EU" device="" value="90"/>
+<part name="R5" library="jack" deviceset="R-EU" device="" value="68"/>
 <part name="GND10" library="cortexm0" deviceset="GND" device=""/>
 <part name="JP3" library="pinhead" deviceset="PINHD-1X8" device=""/>
@@
 <instance part="C7" gate="G$1" x="-19.05" y="-68.58" rot="MR0"/>
 <instance part="GND5" gate="G$1" x="-19.05" y="-73.66"/>
-<instance part="L1" gate="G$1" x="-92.71" y="-87.63"/>
-<instance part="L2" gate="A" x="-35.56" y="-66.04"/>
+<instance part="L1" gate="G$1" x="-92.71" y="-87.63">
+<attribute name="EAGLEUP" x="-92.71" y="-87.63" size="1.27" layer="96" display="off"/>
+</instance>
+<instance part="L2" gate="A" x="-35.56" y="-66.04">
+<attribute name="EAGLEUP" x="-35.56" y="-66.04" size="1.778" layer="96" display="off"/>
+</instance>
 <instance part="J1" gate="G$1" x="-97.79" y="-3.81" rot="MR0"/>
 <instance part="C8" gate="G$1" x="-83.82" y="-15.24"/>
 <instance part="R1" gate="G$1" x="-73.66" y="-17.78" rot="R270"/>
-<instance part="IC1" gate="G$1" x="-62.23" y="-1.27"/>
+<instance part="IC1" gate="G$1" x="-62.23" y="-1.27">
+<attribute name="EAGLEUP" x="-62.23" y="-1.27" size="1.778" layer="96" display="off"/>
+</instance>
 <instance part="GND6" gate="G$1" x="-73.66" y="-25.4"/>
 <instance part="C9" gate="G$1" x="53.34" y="-83.82" rot="MR0"/>
@@
 <instance part="R2" gate="G$1" x="46.99" y="-80.01"/>
 <instance part="R3" gate="G$1" x="53.34" y="-73.66" rot="MR270"/>
-<instance part="SW1" gate="G$1" x="40.64" y="-85.09" rot="R90"/>
-<instance part="IC3" gate="G$1" x="-73.66" y="-50.8"/>
+<instance part="SW1" gate="G$1" x="40.64" y="-85.09" rot="R90">
+<attribute name="EAGLEUP" x="40.64" y="-85.09" size="1.778" layer="96" rot="R90" display="off"/>
+</instance>
+<instance part="IC3" gate="G$1" x="-73.66" y="-50.8">
+<attribute name="EAGLEUP" x="-73.66" y="-50.8" size="1.27" layer="96" display="off"/>
+</instance>
 <instance part="VDD4" gate="G$1" x="-57.15" y="-49.53"/>
 <instance part="VBUS2" gate="G$1" x="-90.17" y="-41.91"/>
@@
 <instance part="C10" gate="G$1" x="-90.17" y="-57.15" rot="MR0"/>
 <instance part="C11" gate="G$1" x="-57.15" y="-57.15"/>
-<instance part="X1" gate="G$1" x="83.82" y="-81.28"/>
+<instance part="X1" gate="G$1" x="83.82" y="-81.28">
+<attribute name="EAGLEUP" x="83.82" y="-81.28" size="1.778" layer="96" display="off"/>
+</instance>
 <instance part="C12" gate="G$1" x="74.93" y="-85.09" rot="MR0"/>
 <instance part="C13" gate="G$1" x="92.71" y="-85.09"/>
 <instance part="GND9" gate="G$1" x="83.82" y="-91.44"/>
-<instance part="D1" gate="G$1" x="-90.17" y="-46.99" rot="R270"/>
-<instance part="D2" gate="G$1" x="-97.79" y="-46.99" rot="R270"/>
+<instance part="D1" gate="G$1" x="-90.17" y="-46.99" rot="R270">
+<attribute name="EAGLEUP" x="-90.17" y="-46.99" size="1.27" layer="96" rot="R270" display="off"/>
+</instance>
+<instance part="D2" gate="G$1" x="-97.79" y="-46.99" rot="R270">
+<attribute name="EAGLEUP" x="-97.79" y="-46.99" size="1.27" layer="96" rot="R270" display="off"/>
+</instance>
 <instance part="U$1" gate="G$1" x="-71.12" y="-99.06"/>
 <instance part="VDD5" gate="G$1" x="-36.83" y="-64.77"/>

Commit message: Updated BOM, JACK logo package, GERBERS, licence, readme
Other:
- note added: "Copyright © Michele Perla 2015 This documentation describes Open Hardware and is licensed under the CERN OHL v. 1.2. You may redistribute and modify this documentation under the terms of the CERN OHL v.1.2. (http://ohwr.org/cernohl). This documentation is distributed WITHOUT ANY EXPRESS OR IMPLIED WARRANTY, INCLUDING OF MERCHANTABILITY, SATISFACTORY QUALITY AND FITNESS FOR A PARTICULAR PURPOSE. P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"
Changed lines of the file:
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@@
 <wire x1="64.77" y1="-97.79" x2="101.6" y2="-97.79" width="0.1524" layer="97" style="shortdash"/>
 <wire x1="64.77" y1="-97.79" x2="64.77" y2="-54.61" width="0.1524" layer="97" style="shortdash"/>
+<text x="149.86" y="-93.98" size="1.778" layer="97">Copyright © Michele Perla 2015
+This documentation describes Open Hardware and is licensed
+under the CERN OHL v. 1.2. You may redistribute and modify
+this documentation under the terms of the CERN OHL v.1.2.
+(http://ohwr.org/cernohl). This documentation is distributed
+WITHOUT ANY EXPRESS OR IMPLIED WARRANTY, INCLUDING
+OF MERCHANTABILITY, SATISFACTORY QUALITY AND FITNESS
+FOR A PARTICULAR PURPOSE. Please see the CERN OHL v.1.2
+for applicable conditions.</text>
 </plain>
 <instances>
